Commit message: Changed joints 1-6 to revolute with -30,30 limits

File: jaco_model/urdf/jaco_arm.xacro (robot description, xacro)
@@ -89,5 +89,5 @@
 </link>
 </xacro:macro>
-<xacro:macro name="jaco_joint" params="joint_name type parent child joint_axis_xyz joint_origin_xyz joint_origin_rpy">
+<xacro:macro name="jaco_joint" params="joint_name type parent child joint_axis_xyz joint_origin_xyz joint_origin_rpy lower_limit upper_limit">
 <joint name="${joint_name}" type="${type}">
     <parent link="${parent}"/>
@@ -95,4 +95,5 @@
     <axis xyz="${joint_axis_xyz}"/>
 <origin xyz="${joint_origin_xyz}" rpy="${joint_origin_rpy}"/>
+ <limit lower="${lower_limit}" upper="${upper_limit}" effort="30" velocity="5"/>
  </joint>
 </xacro:macro>
@@ -108,17 +109,17 @@
 <xacro:macro name="jaco_arm" params="parent">
    <xacro:jaco_link link_name="${link_base}"/>
-   <xacro:jaco_joint joint_name="${joint_base}" type="fixed" parent="${parent}" child="${link_base}" joint_axis_xyz="${joint_base_axis_xyz}" joint_origin_xyz="${joint_base_origin_xyz}" joint_origin_rpy="${joint_base_origin_rpy}"/>
+   <xacro:jaco_joint joint_name="${joint_base}" type="fixed" parent="${parent}" child="${link_base}" joint_axis_xyz="${joint_base_axis_xyz}" joint_origin_xyz="${joint_base_origin_xyz}" joint_origin_rpy="${joint_base_origin_rpy}" lower_limit="-30" upper_limit="30"/>
    <xacro:jaco_link link_name="${link_1}"/>
-   <xacro:jaco_joint joint_name="${joint_1}" type="continuous" parent="${link_base}" child="${link_1}" joint_axis_xyz="${joint_1_axis_xyz}" joint_origin_xyz="${joint_1_origin_xyz}" joint_origin_rpy="${joint_1_origin_rpy}"/>
+   <xacro:jaco_joint joint_name="${joint_1}" type="revolute" parent="${link_base}" child="${link_1}" joint_axis_xyz="${joint_1_axis_xyz}" joint_origin_xyz="${joint_1_origin_xyz}" joint_origin_rpy="${joint_1_origin_rpy}" lower_limit="-30" upper_limit="30"/>
    <xacro:jaco_link link_name="${link_2}"/>
-   <xacro:jaco_joint joint_name="${joint_2}" type="continuous" parent="${link_1}" child="${link_2}" joint_axis_xyz="${joint_2_axis_xyz}" joint_origin_xyz="${joint_2_origin_xyz}" joint_origin_rpy="${joint_2_origin_rpy}"/>
+   <xacro:jaco_joint joint_name="${joint_2}" type="revolute" parent="${link_1}" child="${link_2}" joint_axis_xyz="${joint_2_axis_xyz}" joint_origin_xyz="${joint_2_origin_xyz}" joint_origin_rpy="${joint_2_origin_rpy}" lower_limit="-30" upper_limit="30"/>
    <xacro:jaco_link link_name="${link_3}"/>
-   <xacro:jaco_joint joint_name="${joint_3}" type="continuous" parent="${link_2}" child="${link_3}" joint_axis_xyz="${joint_3_axis_xyz}" joint_origin_xyz="${joint_3_origin_xyz}" joint_origin_rpy="${joint_3_origin_rpy}"/>
+   <xacro:jaco_joint joint_name="${joint_3}" type="revolute" parent="${link_2}" child="${link_3}" joint_axis_xyz="${joint_3_axis_xyz}" joint_origin_xyz="${joint_3_origin_xyz}" joint_origin_rpy="${joint_3_origin_rpy}" lower_limit="-30" upper_limit="30"/>
    <xacro:jaco_link link_name="${link_4}"/>
-   <xacro:jaco_joint joint_name="${joint_4}" type="continuous" parent="${link_3}" child="${link_4}" joint_axis_xyz="${joint_4_axis_xyz}" joint_origin_xyz="${joint_4_origin_xyz}" joint_origin_rpy="${joint_4_origin_rpy}"/>
+   <xacro:jaco_joint joint_name="${joint_4}" type="revolute" parent="${link_3}" child="${link_4}" joint_axis_xyz="${joint_4_axis_xyz}" joint_origin_xyz="${joint_4_origin_xyz}" joint_origin_rpy="${joint_4_origin_rpy}" lower_limit="-30" upper_limit="30"/>
    <xacro:jaco_link link_name="${link_5}"/>
-   <xacro:jaco_joint joint_name="${joint_5}" type="continuous" parent="${link_4}" child="${link_5}" joint_axis_xyz="${joint_5_axis_xyz}" joint_origin_xyz="${joint_5_origin_xyz}" joint_origin_rpy="${joint_5_origin_rpy}"/>
+   <xacro:jaco_joint joint_name="${joint_5}" type="revolute" parent="${link_4}" child="${link_5}" joint_axis_xyz="${joint_5_axis_xyz}" joint_origin_xyz="${joint_5_origin_xyz}" joint_origin_rpy="${joint_5_origin_rpy}" lower_limit="-30" upper_limit="30"/>
    <xacro:jaco_link link_name="${link_hand}"/>
-   <xacro:jaco_joint joint_name="${joint_6}" type="continuous" parent="${link_5}" child="${link_hand}" joint_axis_xyz="${joint_6_axis_xyz}" joint_origin_xyz="${joint_6_origin_xyz}" joint_origin_rpy="${joint_6_origin_rpy}"/>
+   <xacro:jaco_joint joint_name="${joint_6}" type="revolute" parent="${link_5}" child="${link_hand}" joint_axis_xyz="${joint_6_axis_xyz}" joint_origin_xyz="${joint_6_origin_xyz}" joint_origin_rpy="${joint_6_origin_rpy}" lower_limit="-30" upper_limit="30"/>
    <xacro:jaco_link link_name="${link_finger_1}"/>
    <xacro:jaco_finger_joint joint_name="${joint_finger_1}" type="revolute" parent="${link_hand}" child="${link_finger_1}" joint_axis_xyz="${joint_finger_1_axis_xyz}" joint_origin_xyz="${joint_finger_1_origin_xyz}" joint_origin_rpy="${joint_finger_1_origin_rpy}" lower_limit="${joint_finger_1_lower_limit}" upper_limit="${joint_finger_1_upper_limit}"/>

Commit message: Changed joint angle parameters in jaco_arm.xacro

File: jaco_model/urdf/jaco_arm.xacro (robot description, xacro)
@@ -13,44 +13,72 @@
     xmlns:physics="http://playerstage.sourceforge.net/gazebo/xmlschema/#physics"
 	xmlns:xacro="http://ros.org/wiki/xacro">
-  <property name="J_PI" value="3.1415926535897931" />
-  <property name="link_base" value="jaco_link_base" />
-  <property name="link_1" value="jaco_link_1" />
-  <property name="link_2" value="jaco_link_2" />
-  <property name="link_3" value="jaco_link_3" />
-  <property name="link_4" value="jaco_link_4" />
-  <property name="link_5" value="jaco_link_5" />
-  <property name="link_hand" value="jaco_link_hand" />
-  <property name="link_finger_1" value="jaco_link_finger_1" />
-  <property name="link_finger_2" value="jaco_link_finger_2" />
-  <property name="link_finger_3" value="jaco_link_finger_3" />
-  <property name="joint_base" value="jaco_joint_base" />
+  <property name="robot_prefix" value="jaco_"/>
+  <property name="J_PI" value="3.1415926535897932" />
+  <property name="continuous_joint_limit" value="55.55555555555555555555556" />
+  <property name="link_base" value="${robot_prefix}link_base" />
+  <property name="link_1" value="${robot_prefix}link_1" />
+  <property name="link_2" value="${robot_prefix}link_2" />
+  <property name="link_3" value="${robot_prefix}link_3" />
+  <property name="link_4" value="${robot_prefix}link_4" />
+  <property name="link_5" value="${robot_prefix}link_5" />
+  <property name="link_hand" value="${robot_prefix}link_hand" />
+  <property name="link_finger_1" value="${robot_prefix}link_finger_1" />
+  <property name="link_finger_2" value="${robot_prefix}link_finger_2" />
+  <property name="link_finger_3" value="${robot_prefix}link_finger_3" />
+  <property name="joint_base" value="${robot_prefix}joint_base" />
   <property name="joint_base_axis_xyz" value="0 0 0" />
   <property name="joint_base_origin_xyz" value="0 0 0" />
   <property name="joint_base_origin_rpy" value="0 0 0" />
-  <property name="joint_1" value="jaco_joint_1" />
-  <property name="joint_1_axis_xyz" value="0 0 1" />
+  <property name="joint_1" value="${robot_prefix}joint_1" />
+  <property name="joint_1_axis_xyz" value="0 0 -1" />
   <property name="joint_1_origin_xyz" value="0 0 0.1535" />
-  <property name="joint_1_origin_rpy" value="${J_PI} 0 0" />
-  <property name="joint_2" value="jaco_joint_2" />
+  <property name="joint_1_origin_rpy" value="${J_PI} 0 ${J_PI}" />
+  <property name="joint_1_lower_limit" value="-${continuous_joint_limit*J_PI}" />
+  <property name="joint_1_upper_limit" value="${continuous_joint_limit*J_PI}" />
+  <property name="joint_2" value="${robot_prefix}joint_2" />
   <property name="joint_2_axis_xyz" value="0 0 1" />
   <property name="joint_2_origin_xyz" value="0 0 -0.1185" />
-  <property name="joint_2_origin_rpy" value="-${J_PI/2} -${J_PI/2} 0" />
-  <property name="joint_3" value="jaco_joint_3" />
-  <property name="joint_3_axis_xyz" value="0 0 1" />
+  <property name="joint_2_origin_rpy" value="-${J_PI/2} ${J_PI} 0" />
+<!--  <property name="joint_2_origin_xyz" value="0 0 -0.1185" />
+  <property name="joint_2_origin_rpy" value="-${J_PI/2} -${J_PI/2} 0" />-->
+  <property name="joint_2_lower_limit" value="${42*J_PI/180}" />
+  <property name="joint_2_upper_limit" value="${318*J_PI/180}" />
+  <property name="joint_3" value="${robot_prefix}joint_3" />
+<!--  <property name="joint_3_axis_xyz" value="0 0 -1" />
+ <property name="joint_3_origin_xyz" value="0.41 0 0" />
+  <property name="joint_3_origin_rpy" value="${J_PI} 0 ${J_PI/2}" />  -->
+  <property name="joint_3_axis_xyz" value="0 0 -1" />
   <property name="joint_3_origin_xyz" value="0.41 0 0" />
-  <property name="joint_3_origin_rpy" value="${J_PI} 0 ${J_PI}" />
-  <property name="joint_4" value="jaco_joint_4" />
-  <property name="joint_4_axis_xyz" value="0 0 1" />
+  <property name="joint_3_origin_rpy" value="${J_PI} 0 ${J_PI/2}" />
+  <property name="joint_3_lower_limit" value="${17*J_PI/180}" />
+  <property name="joint_3_upper_limit" value="${343*J_PI/180}" />
+  <property name="joint_4" value="${robot_prefix}joint_4" />
+<!-- <property name="joint_4_axis_xyz" value="0 0 -1" />
   <property name="joint_4_origin_xyz" value="0.207 0 -0.01125" />
-  <property name="joint_4_origin_rpy" value="0 -${J_PI/2} 0" />
-  <property name="joint_5" value="jaco_joint_5" />
-  <property name="joint_5_axis_xyz" value="0 0 1" />
+  <property name="joint_4_origin_rpy" value="0 -${J_PI/2} -${J_PI}" /> -->
+  <property name="joint_4_axis_xyz" value="0 0 -1" />
+  <property name="joint_4_origin_xyz" value="0.207 0 -0.01125" />
+  <property name="joint_4_origin_rpy" value="${J_PI} ${J_PI/2} 0" />
+  <property name="joint_4_lower_limit" value="-${continuous_joint_limit*J_PI}" />
+  <property name="joint_4_upper_limit" value="${continuous_joint_limit*J_PI}" />
+  <property name="joint_5" value="${robot_prefix}joint_5" />
+<!-- <property name="joint_5_axis_xyz" value="0 0 -1" />
   <property name="joint_5_origin_xyz" value="0.0343 0 -0.06588" />
-  <property name="joint_5_origin_rpy" value="0 ${J_PI/180*55} ${J_PI}" />
-  <property name="joint_6" value="jaco_joint_6" />
-  <property name="joint_6_axis_xyz" value="0 0 1" />
+  <property name="joint_5_origin_rpy" value="0 ${J_PI/180*55} 0" />  -->
+  <property name="joint_5_axis_xyz" value="0 0 -1" />
+  <property name="joint_5_origin_xyz" value="0.0343 0 -0.06588" />
+  <property name="joint_5_origin_rpy" value="${J_PI} -${J_PI/180*125} ${J_PI}" />
+  <property name="joint_5_lower_limit" value="-${continuous_joint_limit*J_PI}" />
+  <property name="joint_5_upper_limit" value="${continuous_joint_limit*J_PI}" />
+  <property name="joint_6" value="${robot_prefix}joint_6" />
+<!--  <property name="joint_6_axis_xyz" value="0 0 -1" />
   <property name="joint_6_origin_xyz" value="0.0343 0 -0.06588" />
-  <property name="joint_6_origin_rpy" value="0 ${J_PI/180*55} ${J_PI}" />
-  <property name="joint_finger_1" value="jaco_joint_finger_1" />
+  <property name="joint_6_origin_rpy" value="0 ${J_PI/180*55} -${4*J_PI/9}" /> -->
+  <property name="joint_6_axis_xyz" value="0 0 -1" />
+  <property name="joint_6_origin_xyz" value="0.0343 0 -0.06588" />
+  <property name="joint_6_origin_rpy" value="${J_PI} -${J_PI/180*125} ${J_PI}" />
+  <property name="joint_6_lower_limit" value="-${continuous_joint_limit*J_PI}" />
+  <property name="joint_6_upper_limit" value="${continuous_joint_limit*J_PI}" />
+  <property name="joint_finger_1" value="${robot_prefix}joint_finger_1" />
   <property name="joint_finger_1_axis_xyz" value="0 0 1" />
   <property name="joint_finger_1_origin_xyz" value="-0.03978 0 -0.10071" />
@@ -58,5 +86,5 @@
   <property name="joint_finger_1_lower_limit" value="0" />
   <property name="joint_finger_1_upper_limit" value="${J_PI/180*40}" />
-  <property name="joint_finger_2" value="jaco_joint_finger_2" />
+  <property name="joint_finger_2" value="${robot_prefix}joint_finger_2" />
   <property name="joint_finger_2_axis_xyz" value="0 0 1" />
   <property name="joint_finger_2_origin_xyz" value="0.03569 -0.0216 -0.10071" />
@@ -64,5 +92,5 @@
   <property name="joint_finger_2_lower_limit" value="0" />
   <property name="joint_finger_2_upper_limit" value="${J_PI/180*40}" />
-  <property name="joint_finger_3" value="jaco_joint_finger_3" />
+  <property name="joint_finger_3" value="${robot_prefix}joint_finger_3" />
   <property name="joint_finger_3_axis_xyz" value="0 0 1" />
   <property name="joint_finger_3_origin_xyz" value="0.03569 0.0216 -0.10071" />
@@ -89,5 +117,13 @@
 </link>
 </xacro:macro>
-<xacro:macro name="jaco_joint" params="joint_name type parent child joint_axis_xyz joint_origin_xyz joint_origin_rpy">
+<xacro:macro name="jaco_fixed_joint" params="joint_name type parent child joint_axis_xyz joint_origin_xyz joint_origin_rpy">
+<joint name="${joint_name}" type="${type}">
+  <parent link="${parent}"/>
+    <child link="${child}"/>
+    <axis xyz="${joint_axis_xyz}"/>
+    <origin xyz="${joint_origin_xyz}" rpy="${joint_origin_rpy}"/>
+ </joint>
+</xacro:macro>
+<xacro:macro name="jaco_joint" params="joint_name type parent child joint_axis_xyz joint_origin_xyz joint_origin_rpy lower_limit upper_limit">
 <joint name="${joint_name}" type="${type}">
     <parent link="${parent}"/>
@@ -95,4 +131,5 @@
     <axis xyz="${joint_axis_xyz}"/>
 <origin xyz="${joint_origin_xyz}" rpy="${joint_origin_rpy}"/>
+    <limit lower="${lower_limit}" upper="${upper_limit}" effort="30" velocity="5"/>
  </joint>
 </xacro:macro>
@@ -108,17 +145,17 @@
 <xacro:macro name="jaco_arm" params="parent">
    <xacro:jaco_link link_name="${link_base}"/>
-   <xacro:jaco_joint joint_name="${joint_base}" type="fixed" parent="${parent}" child="${link_base}" joint_axis_xyz="${joint_base_axis_xyz}" joint_origin_xyz="${joint_base_origin_xyz}" joint_origin_rpy="${joint_base_origin_rpy}"/>
+   <xacro:jaco_fixed_joint joint_name="${joint_base}" type="fixed" parent="${parent}" child="${link_base}" joint_axis_xyz="${joint_base_axis_xyz}" joint_origin_xyz="${joint_base_origin_xyz}" joint_origin_rpy="${joint_base_origin_rpy}"/>
    <xacro:jaco_link link_name="${link_1}"/>
-   <xacro:jaco_joint joint_name="${joint_1}" type="continuous" parent="${link_base}" child="${link_1}" joint_axis_xyz="${joint_1_axis_xyz}" joint_origin_xyz="${joint_1_origin_xyz}" joint_origin_rpy="${joint_1_origin_rpy}"/>
+   <xacro:jaco_joint joint_name="${joint_1}" type="revolute" parent="${link_base}" child="${link_1}" joint_axis_xyz="${joint_1_axis_xyz}" joint_origin_xyz="${joint_1_origin_xyz}" joint_origin_rpy="${joint_1_origin_rpy}" lower_limit="${joint_1_lower_limit}" upper_limit="${joint_1_upper_limit}"/>
    <xacro:jaco_link link_name="${link_2}"/>
-   <xacro:jaco_joint joint_name="${joint_2}" type="continuous" parent="${link_1}" child="${link_2}" joint_axis_xyz="${joint_2_axis_xyz}" joint_origin_xyz="${joint_2_origin_xyz}" joint_origin_rpy="${joint_2_origin_rpy}"/>
+   <xacro:jaco_joint joint_name="${joint_2}" type="revolute" parent="${link_1}" child="${link_2}" joint_axis_xyz="${joint_2_axis_xyz}" joint_origin_xyz="${joint_2_origin_xyz}" joint_origin_rpy="${joint_2_origin_rpy}" lower_limit="${joint_2_lower_limit}" upper_limit="${joint_2_upper_limit}"/>
    <xacro:jaco_link link_name="${link_3}"/>
-   <xacro:jaco_joint joint_name="${joint_3}" type="continuous" parent="${link_2}" child="${link_3}" joint_axis_xyz="${joint_3_axis_xyz}" joint_origin_xyz="${joint_3_origin_xyz}" joint_origin_rpy="${joint_3_origin_rpy}"/>
+   <xacro:jaco_joint joint_name="${joint_3}" type="revolute" parent="${link_2}" child="${link_3}" joint_axis_xyz="${joint_3_axis_xyz}" joint_origin_xyz="${joint_3_origin_xyz}" joint_origin_rpy="${joint_3_origin_rpy}"  lower_limit="${joint_3_lower_limit}" upper_limit="${joint_3_upper_limit}"/>
    <xacro:jaco_link link_name="${link_4}"/>
-   <xacro:jaco_joint joint_name="${joint_4}" type="continuous" parent="${link_3}" child="${link_4}" joint_axis_xyz="${joint_4_axis_xyz}" joint_origin_xyz="${joint_4_origin_xyz}" joint_origin_rpy="${joint_4_origin_rpy}"/>
+   <xacro:jaco_joint joint_name="${joint_4}" type="revolute" parent="${link_3}" child="${link_4}" joint_axis_xyz="${joint_4_axis_xyz}" joint_origin_xyz="${joint_4_origin_xyz}" joint_origin_rpy="${joint_4_origin_rpy}"  lower_limit="${joint_4_lower_limit}" upper_limit="${joint_4_upper_limit}"/>
    <xacro:jaco_link link_name="${link_5}"/>
-   <xacro:jaco_joint joint_name="${joint_5}" type="continuous" parent="${link_4}" child="${link_5}" joint_axis_xyz="${joint_5_axis_xyz}" joint_origin_xyz="${joint_5_origin_xyz}" joint_origin_rpy="${joint_5_origin_rpy}"/>
+   <xacro:jaco_joint joint_name="${joint_5}" type="revolute" parent="${link_4}" child="${link_5}" joint_axis_xyz="${joint_5_axis_xyz}" joint_origin_xyz="${joint_5_origin_xyz}" joint_origin_rpy="${joint_5_origin_rpy}" lower_limit="${joint_5_lower_limit}" upper_limit="${joint_5_upper_limit}"/>
    <xacro:jaco_link link_name="${link_hand}"/>
-   <xacro:jaco_joint joint_name="${joint_6}" type="continuous" parent="${link_5}" child="${link_hand}" joint_axis_xyz="${joint_6_axis_xyz}" joint_origin_xyz="${joint_6_origin_xyz}" joint_origin_rpy="${joint_6_origin_rpy}"/>
+   <xacro:jaco_joint joint_name="${joint_6}" type="revolute" parent="${link_5}" child="${link_hand}" joint_axis_xyz="${joint_6_axis_xyz}" joint_origin_xyz="${joint_6_origin_xyz}" joint_origin_rpy="${joint_6_origin_rpy}" lower_limit="${joint_6_lower_limit}" upper_limit="${joint_6_upper_limit}"/>
    <xacro:jaco_link link_name="${link_finger_1}"/>
    <xacro:jaco_finger_joint joint_name="${joint_finger_1}" type="revolute" parent="${link_hand}" child="${link_finger_1}" joint_axis_xyz="${joint_finger_1_axis_xyz}" joint_origin_xyz="${joint_finger_1_origin_xyz}" joint_origin_rpy="${joint_finger_1_origin_rpy}" lower_limit="${joint_finger_1_lower_limit}" upper_limit="${joint_finger_1_upper_limit}"/>

File: jaco_model/urdf/standalone_arm.urdf (robot description, URDF)
Before this commit: robot jaco, 11 links, 10 joints
Joints:
- joint jaco_joint_1: axis 0 0 1 -> 0 0 -1; limit (none) -> lower=-174.532925199 upper=174.532925199 effort=30 velocity=5; origin xyz=0 0 0.1535 rpy=3.14159265359 0 0 -> xyz=0 0 0.1535 rpy=3.14159265359 0 -3.14159265359; type continuous -> revolute
- joint jaco_joint_2: limit (none) -> lower=0.733038285838 upper=5.55014702134 effort=30 velocity=5; origin xyz=0 0 -0.1185 rpy=-1.57079632679 -1.57079632679 0 -> xyz=0 0 -0.1185 rpy=-1.57079632679 -1.57079632679 4.71238898038; type continuous -> revolute
- joint jaco_joint_3: axis 0 0 1 -> 0 0 -1; limit (none) -> lower=0.296705972839 upper=5.98647933434 effort=30 velocity=5; origin xyz=0.41 0 0 rpy=3.14159265359 0 3.14159265359 -> xyz=0.41 0 0 rpy=3.14159265359 0 1.57079632679; type continuous -> revolute
- joint jaco_joint_4: axis 0 0 1 -> 0 0 -1; limit (none) -> lower=-174.532925199 upper=174.532925199 effort=30 velocity=5; origin xyz=0.207 0 -0.01125 rpy=0 -1.57079632679 0 -> xyz=0.207 0 -0.01125 rpy=0 -1.57079632679 -3.14159265359; type continuous -> revolute
- joint jaco_joint_5: axis 0 0 1 -> 0 0 -1; limit (none) -> lower=-174.532925199 upper=174.532925199 effort=30 velocity=5; origin xyz=0.0343 0 -0.06588 rpy=0 0.959931088597 3.14159265359 -> xyz=0.0343 0 -0.06588 rpy=0 0.959931088597 0; type continuous -> revolute
- joint jaco_joint_6: axis 0 0 1 -> 0 0 -1; limit (none) -> lower=-174.532925199 upper=174.532925199 effort=30 velocity=5; origin xyz=0.0343 0 -0.06588 rpy=0 0.959931088597 3.14159265359 -> xyz=0.0343 0 -0.06588 rpy=0 0.959931088597 -1.3962634016; type continuous -> revolute
